Commit message: Changed to ROS2 Jazzy

File: champ/champ_description/urdf/leg.urdf.xacro (robot description, xacro)
@@ -139,5 +139,5 @@
         <ros2_control name="${leg}" type="system">
             <hardware>
-                <plugin>gazebo_ros2_control/GazeboSystem</plugin>
+                <plugin>gz_ros2_control/GazeboSimSystem</plugin>
             </hardware>
             <joint name="${leg}_hip_joint">

File: robots/descriptions/go2_description/xacro/gazebo.xacro (robot description, xacro)
@@ -2,19 +2,17 @@
 <robot>
     <gazebo>
-      <plugin name="p3d_base_controller" filename="libgazebo_ros_p3d.so">
-        <ros>
-            <remapping>odom:=odom/ground_truth</remapping>
-        </ros>
-        <body_name>base_link</body_name>
-        <frame_name>world</frame_name>
-        <update_rate>10.0</update_rate>
+      <plugin filename="gz-sim-odometry-publisher-system" name="gz::sim::systems::OdometryPublisher">
+        <odom_frame>world</odom_frame>
+        <robot_base_frame>base_link</robot_base_frame>
+        <odom_publish_frequency>10.0</odom_publish_frequency>
         <xyz_offset>0 0 0</xyz_offset>
         <rpy_offset>0 0 0</rpy_offset>
-        <gaussian_noise>0.01</gaussian_noise>
-    </plugin>
+      </plugin>
     </gazebo>
     <gazebo>
-        <plugin filename="libgazebo_ros2_control.so" name="gazebo_ros2_control">
+      <plugin filename="gz_ros2_control-system" name="gz_ros2_control::GazeboSimROS2ControlPlugin">
         <parameters>$(find go2_description)/config/ros_control/ros_control.yaml</parameters>
+        <robot_param>robot_description</robot_param>
+        <robot_param_node>robot_state_publisher</robot_param_node>
       </plugin>
     </gazebo>
@@ -23,4 +21,5 @@
             <always_on>true</always_on>
             <update_rate>100</update_rate>
+            <topic>imu/data</topic>
             <imu>
             <angular_velocity>
@@ -65,9 +64,5 @@
             </linear_acceleration>
             </imu>
-            <plugin name="imu_plugin" filename="libgazebo_ros_imu_sensor.so">
-                <ros>
-                    <namespace>imu</namespace>
-                    <remapping>~/out:=data</remapping>
-                </ros>
+            <plugin filename="gz-sim-imu-system" name="gz::sim::systems::Imu">
                 <initial_orientation_as_reference>false</initial_orientation_as_reference>
             </plugin>
@@ -106,10 +101,18 @@
         <mu1>0.2</mu1>
         <mu2>0.2</mu2>
-        <self_collide>1</self_collide>
+        <self_collide>0</self_collide>
+       <sensor name="lf_foot_contact" type="contact">
+         <always_on>true</always_on>
+         <update_rate>25.0</update_rate>
+         <contact>
+           <collision>lf_lower_leg_link_fixed_joint_lump__lf_foot_link_collision_1</collision>
+         </contact>
+         <plugin filename="gz-sim-contact-system" name="gz::sim::systems::Contact" />
+       </sensor>
     </gazebo>
     <gazebo reference="lf_foot_link">
         <mu1>0.6</mu1>
         <mu2>0.6</mu2>
-        <self_collide>1</self_collide>
+        <self_collide>0</self_collide>
         <kp>10000.0</kp>
         <kd>1.0</kd>
@@ -131,4 +134,12 @@
         <mu2>0.2</mu2>
         <self_collide>1</self_collide>
+        <sensor name="rf_foot_contact" type="contact">
+        <always_on>true</always_on>
+        <update_rate>25.0</update_rate>
+        <contact>
+          <collision>rf_lower_leg_link_fixed_joint_lump__rf_foot_link_collision_1</collision>
+        </contact>
+        <plugin filename="gz-sim-contact-system" name="gz::sim::systems::Contact" />
+      </sensor>
     </gazebo>
     <gazebo reference="rf_foot_link">
@@ -155,4 +166,12 @@
         <mu2>0.2</mu2>
         <self_collide>1</self_collide>
+  <sensor name="lh_foot_contact" type="contact">
+    <always_on>true</always_on>
+    <update_rate>25.0</update_rate>
+    <contact>
+      <collision>lh_lower_leg_link_fixed_joint_lump__lh_foot_link_collision_1</collision>
+    </contact>
+    <plugin filename="gz-sim-contact-system" name="gz::sim::systems::Contact" />
+  </sensor>
     </gazebo>
     <gazebo reference="lh_foot_link">
@@ -179,4 +198,12 @@
         <mu2>0.2</mu2>
         <self_collide>1</self_collide>
+       <sensor name="rh_foot_contact" type="contact">
+         <always_on>true</always_on>
+         <update_rate>25.0</update_rate>
+         <contact>
+           <collision>rh_lower_leg_link_fixed_joint_lump__rh_foot_link_collision_1</collision>
+         </contact>
+         <plugin filename="gz-sim-contact-system" name="gz::sim::systems::Contact" />
+       </sensor>
     </gazebo>
     <gazebo reference="rh_foot_link">

File: robots/descriptions/go2_description/xacro/leg.xacro (robot description, xacro)
@@ -128,5 +128,5 @@
             </inertial>
         </link>
-        <joint name="${name}_foot_joint" type="fixed">0
+        <joint name="${name}_foot_joint" type="fixed">
             <origin rpy="0 0 0" xyz="0 0 ${-(calf_length)}"/>
             <parent link="${name}_lower_leg_link"/>
@@ -157,5 +157,5 @@
         <ros2_control name="${name}" type="system">
             <hardware>
-                <plugin>gazebo_ros2_control/GazeboSystem</plugin>
+                <plugin>gz_ros2_control/GazeboSimSystem</plugin>
             </hardware>
             <joint name="${name}_hip_joint">
